File: Diseños Kicad/Nivara Coming soon/Nivara.kicad_sch (KiCad schematic)
At the start: 11 parts, among them J1 Screw_Terminal_01x02, J12 Screw_Terminal_01x04, J13 Screw_Terminal_01x02, J14 Screw_Terminal_01x06, J2 Screw_Terminal_01x04, J3 Screw_Terminal_01x02, J4 Screw_Terminal_01x02, J5 Screw_Terminal_01x03, J6 Screw_Terminal_01x02, J9 Screw_Terminal_01x03

Commit message: UPDATE TAREA
Parts:
- removed J12, J2: Screw_Terminal_01x04, TerminalBlock_Phoenix:TerminalBlock_Phoenix_PT-1,5-4-5.0-H_1x04_P5.00mm_Horizontal, symbol Connector:Screw_Terminal_01x04
- removed J13, J3, J6: Screw_Terminal_01x02, TerminalBlock_Phoenix:TerminalBlock_Phoenix_PT-1,5-2-5.0-H_1x02_P5.00mm_Horizontal, symbol Connector:Screw_Terminal_01x02
- removed J14: Screw_Terminal_01x06, TerminalBlock_Phoenix:TerminalBlock_Phoenix_PT-1,5-6-5.0-H_1x06_P5.00mm_Horizontal, symbol Connector:Screw_Terminal_01x06
- removed J5, J9: Screw_Terminal_01x03, TerminalBlock_Phoenix:TerminalBlock_Phoenix_PT-1,5-3-3.5-H_1x03_P3.50mm_Horizontal, symbol Connector:Screw_Terminal_01x03
- added J10, J11, J2, J5, J9: Screw_Terminal_01x02, symbol Connector:Screw_Terminal_01x02
- added J3: Screw_Terminal_01x04, symbol Connector:Screw_Terminal_01x04
- added J6: Screw_Terminal_01x06, symbol Connector:Screw_Terminal_01x06
- added J7, J8: Screw_Terminal_01x03, symbol Connector:Screw_Terminal_01x03
- AE1: value Wifi -> WIFI-BT
- J1, J4: footprint TerminalBlock_Phoenix:TerminalBlock_Phoenix_PT-1,5-2-5.0-H_1x02_P5.00mm_Horizontal -> (none)
Connections:
- net GND: now also J11.2 (Pin_2), J3.4 (Pin_4), J5.2 (Pin_2), J7.3 (Pin_3), J8.3 (Pin_3)
- net VCC: now also J11.1 (Pin_1)
- net Board_Nivara/D_IN1 renamed NIVARA_BOARD/OPTO_DINPUT_0
- net Board_Nivara/D_IN_2 renamed NIVARA_BOARD/OPTO_DINPUT_1
- net Board_Nivara/NPN_IN_2 renamed NIVARA_BOARD/NPN_DINPUT_0
- net Board_Nivara/NPN_in_1 renamed NIVARA_BOARD/NPN_DINPUT_1
- new net NIVARA_BOARD/+10V_AINPUT: J3.1 (Pin_1)
- new net NIVARA_BOARD/+32V_AINPUT: J3.2 (Pin_2)
- new net NIVARA_BOARD/NPN_DOUTPUT_0: J9.1 (Pin_1)
- new net NIVARA_BOARD/NPN_DOUTPUT_1: J9.2 (Pin_2)
- new net NIVARA_BOARD/PNP_DINPUT_0: J2.1 (Pin_1)
- new net NIVARA_BOARD/PNP_DINPUT_1: J2.2 (Pin_2)
- new net NIVARA_BOARD/PNP_DOUTPUT_0: J10.1 (Pin_1)
- new net NIVARA_BOARD/PNP_DOUTPUT_1: J10.2 (Pin_2)
- new net NIVARA_BOARD/RL1_COM: J6.3 (Pin_3)
- new net NIVARA_BOARD/RL1_OUTPUT_NC: J6.2 (Pin_2)
- new net NIVARA_BOARD/RL1_OUTPUT_NO: J6.1 (Pin_1)
- new net NIVARA_BOARD/RL2_COM: J6.6 (Pin_6)
- new net NIVARA_BOARD/RL2_OUTPUT_NC: J6.5 (Pin_5)
- new net NIVARA_BOARD/RL2_OUTPUT_NO: J6.4 (Pin_4)
- new net NIVARA_BOARD/RS485_A: J7.1 (Pin_1)
- new net NIVARA_BOARD/RS485_B: J7.2 (Pin_2)
- new net NIVARA_BOARD/VOLTAGE_AOUTPUT: J8.1 (Pin_1)
- new net NIVARA_BOARD/mA_AINPUT: J3.3 (Pin_3)
- new net NIVARA_BOARD/mA_AOUTPUT: J8.2 (Pin_2)
- new net NIVARA_BOARD/~{RUN}/STOP: J5.1 (Pin_1)
Other:
- removed sheet Board_Nivara
- added sheet NIVARA_BOARD (NIVARA_BOARD.kicad_sch)
- note added: "+24VDC"
- note removed: "24vdc"
- note removed: "Entrada stop-run"
- company: Electia_ITLA -> (none)
- title: ZorionX-Nivara -> (none)

Commit message: AMEN
Parts:
- AE1: value WIFI-BT -> Antenna
Other:
- moved on the sheet: AE1, J11
Changed lines of the file:
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@@
 	(generator_version "9.0")
 	(paper "A4")
+	(rectangle
+		(start 85.09 91.44)
+		(end 110.49 115.57)
+		(stroke
+			(width 0)
+			(type default)
+		)
+		(fill
+			(type none)
+		)
+	)
 	(text "+24VDC\n"
 		(exclude_from_sim no)
-		(at 141.478 114.554 0)
+		(at 103.378 104.394 0)
 		(effects
 			(font
@@
 	(wire
 		(pts
-			(xy 137.16 113.03) (xy 137.16 111.76)
+			(xy 99.06 102.87) (xy 99.06 101.6)
 		)
 		(stroke
@@
 	(wire
 		(pts
-			(xy 135.89 113.03) (xy 137.16 113.03)
+			(xy 97.79 102.87) (xy 99.06 102.87)
 		)
 		(stroke
@@
 	(wire
 		(pts
-			(xy 135.89 115.57) (xy 137.16 115.57)
+			(xy 97.79 105.41) (xy 99.06 105.41)
 		)
 		(stroke
@@
 	(wire
 		(pts
-			(xy 137.16 115.57) (xy 137.16 116.84)
+			(xy 99.06 105.41) (xy 99.06 106.68)
 		)
 		(stroke
@@
 	(symbol
 		(lib_id "power:VCC")
-		(at 137.16 111.76 0)
+		(at 99.06 101.6 0)
 		(unit 1)
 		(exclude_from_sim no)
@@
 		(dnp no)
 		(fields_autoplaced yes)
-		(property "Reference" "#PWR07"
-			(at 137.16 115.57 0)
+		(property "Reference" "#PWR7"
+			(at 99.06 105.41 0)
 			(effects
 				(font
@@
 		)
 		(property "Value" "VCC"
-			(at 137.16 106.68 0)
-			(effects
-				(font
-					(size 1.27 1.27)
-				)
-			)
-		)
-		(property "Footprint" ""
-			(at 137.16 111.76 0)
+			(at 99.06 96.52 0)
+			(effects
+				(font
+					(size 1.27 1.27)
+				)
+			)
+		)
+		(property "Footprint" ""
+			(at 99.06 101.6 0)
 			(effects
 				(font
@@
 		)
 		(property "Datasheet" ""
-			(at 137.16 111.76 0)
+			(at 99.06 101.6 0)
 			(effects
 				(font
@@
 		)
 		(property "Description" "Power symbol creates a global label with name \"VCC\""
-			(at 137.16 111.76 0)
+			(at 99.06 101.6 0)
 			(effects
 				(font
@@
 			(project ""
 				(path "/8290cc18-06d0-4e02-a781-29a61ebc321a"
-					(reference "#PWR07")
+					(reference "#PWR7")
 					(unit 1)
 				)
@@
 		(dnp no)
 		(fields_autoplaced yes)
-		(property "Reference" "#PWR05"
+		(property "Reference" "#PWR5"
 			(at 184.15 63.5 0)
 			(effects
@@
 			(project "NIVARA"
 				(path "/8290cc18-06d0-4e02-a781-29a61ebc321a"
-					(reference "#PWR05")
+					(reference "#PWR5")
 					(unit 1)
 				)
@@
 		(dnp no)
 		(fields_autoplaced yes)
-		(property "Reference" "#PWR03"
+		(property "Reference" "#PWR3"
 			(at 111.76 87.63 0)
 			(effects
@@
 			(project "NIVARA"
 				(path "/8290cc18-06d0-4e02-a781-29a61ebc321a"
-					(reference "#PWR03")
+					(reference "#PWR3")
 					(unit 1)
 				)
@@
 	(symbol
 		(lib_id "power:GND")
-		(at 137.16 116.84 0)
+		(at 99.06 106.68 0)
 		(unit 1)
 		(exclude_from_sim no)
@@
 		(dnp no)
 		(fields_autoplaced yes)
-		(property "Reference" "#PWR06"
-			(at 137.16 123.19 0)
+		(property "Reference" "#PWR6"
+			(at 99.06 113.03 0)
 			(effects
 				(font
@@
 		)
 		(property "Value" "GND"
-			(at 137.16 121.92 0)
-			(effects
-				(font
-					(size 1.27 1.27)
-				)
-			)
-		)
-		(property "Footprint" ""
-			(at 137.16 116.84 0)
+			(at 99.06 111.76 0)
+			(effects
+				(font
+					(size 1.27 1.27)
+				)
+			)
+		)
+		(property "Footprint" ""
+			(at 99.06 106.68 0)
 			(effects
 				(font
@@
 		)
 		(property "Datasheet" ""
-			(at 137.16 116.84 0)
+			(at 99.06 106.68 0)
 			(effects
 				(font
@@
 		)
 		(property "Description" "Power symbol creates a global label with name \"GND\" , ground"
-			(at 137.16 116.84 0)
+			(at 99.06 106.68 0)
 			(effects
 				(font
@@
 			(project ""
 				(path "/8290cc18-06d0-4e02-a781-29a61ebc321a"
-					(reference "#PWR06")
+					(reference "#PWR6")
 					(unit 1)
 				)
@@
 		(dnp no)
 		(fields_autoplaced yes)
-		(property "Reference" "#PWR04"
+		(property "Reference" "#PWR4"
 			(at 184.15 53.34 0)
 			(effects
@@
 			(project "NIVARA"
 				(path "/8290cc18-06d0-4e02-a781-29a61ebc321a"
-					(reference "#PWR04")
+					(reference "#PWR4")
 					(unit 1)
 				)
@@
 		(dnp no)
 		(fields_autoplaced yes)
-		(property "Reference" "#PWR02"
+		(property "Reference" "#PWR2"
 			(at 111.76 72.39 0)
 			(effects
@@
 			(project ""
 				(path "/8290cc18-06d0-4e02-a781-29a61ebc321a"
-					(reference "#PWR02")
+					(reference "#PWR2")
 					(unit 1)
 				)
@@
 	(symbol
 		(lib_id "Connector:Screw_Terminal_01x02")
-		(at 130.81 113.03 0)
+		(at 92.71 102.87 0)
 		(mirror y)
 		(unit 1)
@@
 		(dnp no)
 		(property "Reference" "J11"
-			(at 130.81 110.49 0)
+			(at 92.71 100.33 0)
 			(effects
 				(font
@@
 		)
 		(property "Value" "Screw_Terminal_01x02"
-			(at 130.81 109.22 0)
-			(effects
-				(font
-					(size 1.27 1.27)
-				)
-				(hide yes)
-			)
-		)
-		(property "Footprint" ""
-			(at 130.81 113.03 0)
+			(at 92.71 99.06 0)
+			(effects
+				(font
+					(size 1.27 1.27)
+				)
+				(hide yes)
+			)
+		)
+		(property "Footprint" ""
+			(at 92.71 102.87 0)
 			(effects
 				(font
@@
 		)
 		(property "Datasheet" "~"
-			(at 130.81 113.03 0)
+			(at 92.71 102.87 0)
 			(effects
 				(font
@@
 		)
 		(property "Description" "Generic screw terminal, single row, 01x02, script generated (kicad-library-utils/schlib/autogen/connector/)"
-			(at 130.81 113.03 0)
+			(at 92.71 102.87 0)
 			(effects
 				(font
@@
 	(symbol
 		(lib_id "Device:Antenna")
-		(at 154.94 115.57 0)
+		(at 116.84 110.49 0)
 		(unit 1)
 		(exclude_from_sim no)
@@
 		(fields_autoplaced yes)
 		(property "Reference" "AE1"
-			(at 157.48 114.9349 0)
+			(at 119.38 109.8549 0)
 			(effects
 				(font
@@
 			)
 		)
-		(property "Value" "WIFI-BT"
-			(at 157.48 117.4749 0)
+		(property "Value" "Antenna"
+			(at 119.38 112.3949 0)
 			(effects
 				(font
@@
 		)
 		(property "Footprint" ""
-			(at 154.94 115.57 0)
+			(at 116.84 110.49 0)
 			(effects
 				(font
@@
 		)
 		(property "Datasheet" "~"
-			(at 154.94 115.57 0)
+			(at 116.84 110.49 0)
 			(effects
 				(font
@@
 		)
 		(property "Description" "Antenna"
-			(at 154.94 115.57 0)
-			(effects
-				(font
+			(at 116.84 110.49 0)
+			(effects
+				(font
