File: Diseños Kicad/NIVARA COMING SOON/NIVARA_BOARD.kicad_sch (KiCad schematic)
At the start: 3 parts, among them U1 ESP32-S3-WROOM-1

Commit message: AMEN
Connections:
- net RELAY_INTERFAZ/RL1_EN: now also U1.38 (GPIO2/TOUCH2/ADC1_CH1)
- net RELAY_INTERFAZ/RL2_EN: now also U1.15 (GPIO3/TOUCH3/ADC1_CH2)
- net mA_INTERFAZ_ENTRADA/mA_READ: now reaches U1.39 (GPIO1/TOUCH1/ADC1_CH0)
- net mA_INTERFAZ_SALIDA/mA_IN: now reaches U1.4 (GPIO4/TOUCH4/ADC1_CH3)
Other:
- sheet RELAY_INTERFACE renamed RELAY_INTERFAZ
- sheet RS485_INTERFACE renamed RS485_INTERFAZ
- added sheet NPN_ENTRADA_Mod (NPN_IN_Mod.kicad_sch)
- added sheet mA_INTERFAZ_ENTRADA (mA_INTERFACE_IN.kicad_sch)
- added sheet mA_INTERFAZ_SALIDA (mA_INTERFACE.kicad_sch)
- sheet RELAY_INTERFAZ ports: added none; removed ST1, ST2
