File: Diseños Kicad/NIVARA COMING SOON/PSU.kicad_sch (KiCad schematic)
At the start: 7 parts, among them U2 AP63203WU

Commit message: AMEN
Parts:
- removed U2: AP63203WU, Package_TO_SOT_SMD:TSOT-23-6, symbol Regulator_Switching:AP63203WU
- added C6: C, symbol Device:C
- added R2, R3: R, symbol Device:R
- added U2: AP63200WU, Package_TO_SOT_SMD:TSOT-23-6, symbol Regulator_Switching:AP63200WU
- C3: Voltage (none) -> 50V
Connections:
- net GND: now also R3.2, U2.4 (GND)
- net VCC: now also U2.2 (EN), U2.3 (IN)
- net at C4.2, C5.2, JP1.1 (A)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: now also C6.1, R2.1
- net at C2.1: now also U2.6 (BST)
- net at C2.2, L1.1: now also U2.5 (SW)
- new net: C6.2, R2.2, R3.1, U2.1 (FB)
Other:
- note added: "AP63200/AP63201 OR AP63203"
- note added: "DO NOT MOUNT FOR AP63203: C6 R3 SUBSITUTE: R2 -> 0Ohm"
