File: Diseños Kicad/NIVARA COMING SOON/RS485_INTERFACE.kicad_sch (KiCad schematic)
At the start: 1 part

Commit message: AMEN
Changed lines of the file:
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@@
 		(dnp no)
 		(fields_autoplaced yes)
-		(property "Reference" "#PWR016"
+		(property "Reference" "#PWR16"
 			(at 116.84 95.25 0)
 			(effects
@@
 			(project ""
 				(path "/8290cc18-06d0-4e02-a781-29a61ebc321a/9e4d7a0c-a5eb-4e88-9036-0c35e68b279a/43a112db-786f-42fb-8db3-67286b51ed8f"
-					(reference "#PWR016")
+					(reference "#PWR16")
 					(unit 1)
 				)
@@
 		(dnp no)
 		(fields_autoplaced yes)
-		(property "Reference" "#PWR017"
+		(property "Reference" "#PWR17"
 			(at 120.65 59.69 0)
 			(effects
@@
 			(project ""
 				(path "/8290cc18-06d0-4e02-a781-29a61ebc321a/9e4d7a0c-a5eb-4e88-9036-0c35e68b279a/43a112db-786f-42fb-8db3-67286b51ed8f"
-					(reference "#PWR017")
+					(reference "#PWR17")
 					(unit 1)
 				)
