File: Diseños Kicad/NIVARA CHECK/10V_AIN_INTERFAZ.kicad_sch (KiCad schematic)
At the start: 3 parts

Commit message: YA AAAAAAAAAAAAAAAA
Detallitos sobre el dxf que estaba mal
Other:
- moved on the sheet: C10, R16, R17
Changed lines of the file:
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@@
 	(paper "A4")
 	(rectangle
-		(start 17.78 15.24)
-		(end 66.04 62.23)
+		(start 16.51 15.24)
+		(end 66.04 60.96)
 		(stroke
 			(width 0)
@@
 	)
 	(junction
-		(at 40.64 44.45)
+		(at 36.83 44.45)
 		(diameter 0)
 		(color 0 0 0 0)
 	)
 	(junction
-		(at 40.64 35.56)
+		(at 36.83 35.56)
 		(diameter 0)
 		(color 0 0 0 0)
 	)
 	(junction
-		(at 49.53 35.56)
+		(at 45.72 35.56)
 		(diameter 0)
 		(color 0 0 0 0)
@@
 	(wire
 		(pts
-			(xy 40.64 33.02) (xy 40.64 35.56)
-		)
-		(stroke
-			(width 0)
-			(type default)
-		)
-	)
-	(wire
-		(pts
-			(xy 49.53 35.56) (xy 54.61 35.56)
-		)
-		(stroke
-			(width 0)
-			(type default)
-		)
-	)
-	(wire
-		(pts
-			(xy 40.64 44.45) (xy 40.64 46.99)
-		)
-		(stroke
-			(width 0)
-			(type default)
-		)
-	)
-	(wire
-		(pts
-			(xy 40.64 22.86) (xy 40.64 25.4)
-		)
-		(stroke
-			(width 0)
-			(type default)
-		)
-	)
-	(wire
-		(pts
-			(xy 49.53 35.56) (xy 49.53 36.83)
-		)
-		(stroke
-			(width 0)
-			(type default)
-		)
-	)
-	(wire
-		(pts
-			(xy 40.64 35.56) (xy 49.53 35.56)
-		)
-		(stroke
-			(width 0)
-			(type default)
-		)
-	)
-	(wire
-		(pts
-			(xy 34.29 22.86) (xy 40.64 22.86)
-		)
-		(stroke
-			(width 0)
-			(type default)
-		)
-	)
-	(wire
-		(pts
-			(xy 40.64 44.45) (xy 49.53 44.45)
-		)
-		(stroke
-			(width 0)
-			(type default)
-		)
-	)
-	(wire
-		(pts
-			(xy 40.64 35.56) (xy 40.64 36.83)
+			(xy 36.83 33.02) (xy 36.83 35.56)
+		)
+		(stroke
+			(width 0)
+			(type default)
+		)
+	)
+	(wire
+		(pts
+			(xy 45.72 35.56) (xy 50.8 35.56)
+		)
+		(stroke
+			(width 0)
+			(type default)
+		)
+	)
+	(wire
+		(pts
+			(xy 36.83 44.45) (xy 36.83 46.99)
+		)
+		(stroke
+			(width 0)
+			(type default)
+		)
+	)
+	(wire
+		(pts
+			(xy 36.83 22.86) (xy 36.83 25.4)
+		)
+		(stroke
+			(width 0)
+			(type default)
+		)
+	)
+	(wire
+		(pts
+			(xy 45.72 35.56) (xy 45.72 36.83)
+		)
+		(stroke
+			(width 0)
+			(type default)
+		)
+	)
+	(wire
+		(pts
+			(xy 36.83 35.56) (xy 45.72 35.56)
+		)
+		(stroke
+			(width 0)
+			(type default)
+		)
+	)
+	(wire
+		(pts
+			(xy 30.48 22.86) (xy 36.83 22.86)
+		)
+		(stroke
+			(width 0)
+			(type default)
+		)
+	)
+	(wire
+		(pts
+			(xy 36.83 44.45) (xy 45.72 44.45)
+		)
+		(stroke
+			(width 0)
+			(type default)
+		)
+	)
+	(wire
+		(pts
+			(xy 36.83 35.56) (xy 36.83 36.83)
 		)
 		(stroke
@@
 	(hierarchical_label "10V_ADC"
 		(shape output)
-		(at 54.61 35.56 0)
+		(at 50.8 35.56 0)
 		(effects
 			(font
@@
 	(hierarchical_label "10V_AIN"
 		(shape input)
-		(at 34.29 22.86 180)
+		(at 30.48 22.86 180)
 		(effects
 			(font
@@
 	(symbol
 		(lib_id "Device:R")
-		(at 40.64 40.64 0)
+		(at 36.83 40.64 0)
 		(unit 1)
 		(exclude_from_sim no)
@@
 		(fields_autoplaced yes)
 		(property "Reference" "R17"
-			(at 43.18 39.3699 0)
+			(at 39.37 39.3699 0)
 			(effects
 				(font
@@
 		)
 		(property "Value" "16k"
-			(at 43.18 41.9099 0)
+			(at 39.37 41.9099 0)
 			(effects
 				(font
@@
 		)
 		(property "Footprint" ""
-			(at 38.862 40.64 90)
+			(at 35.052 40.64 90)
 			(effects
 				(font
@@
 		)
 		(property "Datasheet" "~"
-			(at 40.64 40.64 0)
+			(at 36.83 40.64 0)
 			(effects
 				(font
@@
 		)
 		(property "Description" "Resistor"
-			(at 40.64 40.64 0)
+			(at 36.83 40.64 0)
 			(effects
 				(font
@@
 	(symbol
 		(lib_id "Device:C")
-		(at 49.53 40.64 0)
+		(at 45.72 40.64 0)
 		(unit 1)
 		(exclude_from_sim no)
@@
 		(fields_autoplaced yes)
 		(property "Reference" "C10"
-			(at 53.34 39.3699 0)
+			(at 49.53 39.3699 0)
 			(effects
 				(font
@@
 		)
 		(property "Value" "100nF"
-			(at 53.34 41.9099 0)
+			(at 49.53 41.9099 0)
 			(effects
 				(font
@@
 		)
 		(property "Footprint" ""
-			(at 50.4952 44.45 0)
+			(at 46.6852 44.45 0)
 			(effects
 				(font
@@
 		)
 		(property "Datasheet" "~"
-			(at 49.53 40.64 0)
+			(at 45.72 40.64 0)
 			(effects
 				(font
@@
 		)
 		(property "Description" "Unpolarized capacitor"
-			(at 49.53 40.64 0)
+			(at 45.72 40.64 0)
 			(effects
 				(font
@@
 	(symbol
 		(lib_id "power:GND")
-		(at 40.64 46.99 0)
+		(at 36.83 46.99 0)
 		(unit 1)
 		(exclude_from_sim no)
@@
 		(fields_autoplaced yes)
 		(property "Reference" "#PWR041"
-			(at 40.64 53.34 0)
+			(at 36.83 53.34 0)
 			(effects
 				(font
@@
 		)
 		(property "Value" "GND"
-			(at 40.64 52.07 0)
+			(at 36.83 52.07 0)
 			(effects
 				(font
@@
 		)
 		(property "Footprint" ""
-			(at 40.64 46.99 0)
+			(at 36.83 46.99 0)
 			(effects
 				(font
@@
 		)
 		(property "Datasheet" ""
-			(at 40.64 46.99 0)
+			(at 36.83 46.99 0)
 			(effects
 				(font
@@
 		)
 		(property "Description" "Power symbol creates a global label with name \"GND\" , ground"
-			(at 40.64 46.99 0)
+			(at 36.83 46.99 0)
 			(effects
 				(font
@@
 	(symbol
 		(lib_id "Device:R")
-		(at 40.64 29.21 0)
+		(at 36.83 29.21 0)
 		(unit 1)
 		(exclude_from_sim no)
@@
 		(fields_autoplaced yes)
 		(property "Reference" "R16"
-			(at 43.18 27.9399 0)
+			(at 39.37 27.9399 0)
 			(effects
 				(font
@@
 		)
 		(property "Value" "51k"
-			(at 43.18 30.4799 0)
+			(at 39.37 30.4799 0)
 			(effects
 				(font
@@
 		)
 		(property "Footprint" ""
-			(at 38.862 29.21 90)
+			(at 35.052 29.21 90)
 			(effects
 				(font
@@
 		)
 		(property "Datasheet" "~"
-			(at 40.64 29.21 0)
+			(at 36.83 29.21 0)
 			(effects
 				(font
@@
 		)
 		(property "Description" "Resistor"
-			(at 40.64 29.21 0)
-			(effects
-				(font
+			(at 36.83 29.21 0)
+			(effects
+				(font
