File: Diseños Kicad/NIVARA CHECK/32V_AIN_INTERFAZ.kicad_sch (KiCad schematic)
At the start: 3 parts

Commit message: YA AAAAAAAAAAAAAAAA
Detallitos sobre el dxf que estaba mal
Other:
- moved on the sheet: C9, R14, R15
Changed lines of the file:
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@@
 	(paper "A4")
 	(rectangle
-		(start 17.78 19.05)
-		(end 73.66 67.31)
+		(start 17.78 16.51)
+		(end 64.77 55.88)
 		(stroke
 			(width 0)
@@
 	)
 	(junction
-		(at 41.91 39.37)
+		(at 38.1 31.75)
 		(diameter 0)
 		(color 0 0 0 0)
 	)
 	(junction
-		(at 41.91 48.26)
+		(at 38.1 40.64)
 		(diameter 0)
 		(color 0 0 0 0)
 	)
 	(junction
-		(at 52.07 39.37)
+		(at 48.26 31.75)
 		(diameter 0)
 		(color 0 0 0 0)
@@
 	(wire
 		(pts
-			(xy 41.91 39.37) (xy 41.91 40.64)
-		)
-		(stroke
-			(width 0)
-			(type default)
-		)
-	)
-	(wire
-		(pts
-			(xy 52.07 39.37) (xy 54.61 39.37)
-		)
-		(stroke
-			(width 0)
-			(type default)
-		)
-	)
-	(wire
-		(pts
-			(xy 41.91 48.26) (xy 41.91 50.8)
-		)
-		(stroke
-			(width 0)
-			(type default)
-		)
-	)
-	(wire
-		(pts
-			(xy 41.91 36.83) (xy 41.91 39.37)
-		)
-		(stroke
-			(width 0)
-			(type default)
-		)
-	)
-	(wire
-		(pts
-			(xy 52.07 40.64) (xy 52.07 39.37)
-		)
-		(stroke
-			(width 0)
-			(type default)
-		)
-	)
-	(wire
-		(pts
-			(xy 41.91 39.37) (xy 52.07 39.37)
-		)
-		(stroke
-			(width 0)
-			(type default)
-		)
-	)
-	(wire
-		(pts
-			(xy 41.91 26.67) (xy 41.91 29.21)
-		)
-		(stroke
-			(width 0)
-			(type default)
-		)
-	)
-	(wire
-		(pts
-			(xy 35.56 26.67) (xy 41.91 26.67)
-		)
-		(stroke
-			(width 0)
-			(type default)
-		)
-	)
-	(wire
-		(pts
-			(xy 41.91 48.26) (xy 52.07 48.26)
+			(xy 38.1 31.75) (xy 38.1 33.02)
+		)
+		(stroke
+			(width 0)
+			(type default)
+		)
+	)
+	(wire
+		(pts
+			(xy 48.26 31.75) (xy 50.8 31.75)
+		)
+		(stroke
+			(width 0)
+			(type default)
+		)
+	)
+	(wire
+		(pts
+			(xy 38.1 40.64) (xy 38.1 43.18)
+		)
+		(stroke
+			(width 0)
+			(type default)
+		)
+	)
+	(wire
+		(pts
+			(xy 38.1 29.21) (xy 38.1 31.75)
+		)
+		(stroke
+			(width 0)
+			(type default)
+		)
+	)
+	(wire
+		(pts
+			(xy 48.26 33.02) (xy 48.26 31.75)
+		)
+		(stroke
+			(width 0)
+			(type default)
+		)
+	)
+	(wire
+		(pts
+			(xy 38.1 31.75) (xy 48.26 31.75)
+		)
+		(stroke
+			(width 0)
+			(type default)
+		)
+	)
+	(wire
+		(pts
+			(xy 38.1 19.05) (xy 38.1 21.59)
+		)
+		(stroke
+			(width 0)
+			(type default)
+		)
+	)
+	(wire
+		(pts
+			(xy 31.75 19.05) (xy 38.1 19.05)
+		)
+		(stroke
+			(width 0)
+			(type default)
+		)
+	)
+	(wire
+		(pts
+			(xy 38.1 40.64) (xy 48.26 40.64)
 		)
 		(stroke
@@
 	(hierarchical_label "32V_ADC"
 		(shape output)
-		(at 54.61 39.37 0)
+		(at 50.8 31.75 0)
 		(effects
 			(font
@@
 	(hierarchical_label "32V_AIN"
 		(shape input)
-		(at 35.56 26.67 180)
+		(at 31.75 19.05 180)
 		(effects
 			(font
@@
 	(symbol
 		(lib_id "Device:R")
-		(at 41.91 44.45 0)
+		(at 38.1 36.83 0)
 		(unit 1)
 		(exclude_from_sim no)
@@
 		(fields_autoplaced yes)
 		(property "Reference" "R15"
-			(at 44.45 43.1799 0)
+			(at 40.64 35.5599 0)
 			(effects
 				(font
@@
 		)
 		(property "Value" "13k"
-			(at 44.45 45.7199 0)
+			(at 40.64 38.0999 0)
 			(effects
 				(font
@@
 		)
 		(property "Footprint" ""
-			(at 40.132 44.45 90)
+			(at 36.322 36.83 90)
 			(effects
 				(font
@@
 		)
 		(property "Datasheet" "~"
-			(at 41.91 44.45 0)
+			(at 38.1 36.83 0)
 			(effects
 				(font
@@
 		)
 		(property "Description" "Resistor"
-			(at 41.91 44.45 0)
+			(at 38.1 36.83 0)
 			(effects
 				(font
@@
 	(symbol
 		(lib_id "Device:C")
-		(at 52.07 44.45 0)
+		(at 48.26 36.83 0)
 		(unit 1)
 		(exclude_from_sim no)
@@
 		(fields_autoplaced yes)
 		(property "Reference" "C9"
-			(at 55.88 43.1799 0)
+			(at 52.07 35.5599 0)
 			(effects
 				(font
@@
 		)
 		(property "Value" "100nF"
-			(at 55.88 45.7199 0)
+			(at 52.07 38.0999 0)
 			(effects
 				(font
@@
 		)
 		(property "Footprint" ""
-			(at 53.0352 48.26 0)
+			(at 49.2252 40.64 0)
 			(effects
 				(font
@@
 		)
 		(property "Datasheet" "~"
-			(at 52.07 44.45 0)
+			(at 48.26 36.83 0)
 			(effects
 				(font
@@
 		)
 		(property "Description" "Unpolarized capacitor"
-			(at 52.07 44.45 0)
+			(at 48.26 36.83 0)
 			(effects
 				(font
@@
 	(symbol
 		(lib_id "power:GND")
-		(at 41.91 50.8 0)
+		(at 38.1 43.18 0)
 		(unit 1)
 		(exclude_from_sim no)
@@
 		(fields_autoplaced yes)
 		(property "Reference" "#PWR038"
-			(at 41.91 57.15 0)
+			(at 38.1 49.53 0)
 			(effects
 				(font
@@
 		)
 		(property "Value" "GND"
-			(at 41.91 55.88 0)
+			(at 38.1 48.26 0)
 			(effects
 				(font
@@
 		)
 		(property "Footprint" ""
-			(at 41.91 50.8 0)
+			(at 38.1 43.18 0)
 			(effects
 				(font
@@
 		)
 		(property "Datasheet" ""
-			(at 41.91 50.8 0)
+			(at 38.1 43.18 0)
 			(effects
 				(font
@@
 		)
 		(property "Description" "Power symbol creates a global label with name \"GND\" , ground"
-			(at 41.91 50.8 0)
+			(at 38.1 43.18 0)
 			(effects
 				(font
@@
 	(symbol
 		(lib_id "Device:R")
-		(at 41.91 33.02 0)
+		(at 38.1 25.4 0)
 		(unit 1)
 		(exclude_from_sim no)
@@
 		(fields_autoplaced yes)
 		(property "Reference" "R14"
-			(at 44.45 31.7499 0)
+			(at 40.64 24.1299 0)
 			(effects
 				(font
@@
 		)
 		(property "Value" "160k"
-			(at 44.45 34.2899 0)
+			(at 40.64 26.6699 0)
 			(effects
 				(font
@@
 		)
 		(property "Footprint" ""
-			(at 40.132 33.02 90)
+			(at 36.322 25.4 90)
 			(effects
 				(font
@@
 		)
 		(property "Datasheet" "~"
-			(at 41.91 33.02 0)
+			(at 38.1 25.4 0)
 			(effects
 				(font
@@
 		)
 		(property "Description" "Resistor"
-			(at 41.91 33.02 0)
-			(effects
-				(font
+			(at 38.1 25.4 0)
+			(effects
+				(font
