File: Diseños Kicad/NIVARA CHECK/DRY_INPUT_INTERFAZ.kicad_sch (KiCad schematic)
At the start: 6 parts, among them U7 LTV-357TB, U8 LTV-357TB

Commit message: YA AAAAAAAAAAAAAAAA
Detallitos sobre el dxf que estaba mal
Other:
- moved on the sheet: R10, R11, R12, R13, U7, U8
