File: Diseños Kicad/NIVARA CHECK/NIVARA.kicad_sch (KiCad schematic)
At the start: 12 parts, among them J1 Screw_Terminal_01x02, J10 Screw_Terminal_01x02, J11 Screw_Terminal_01x02, J12 Screw_Terminal_01x04, J2 Screw_Terminal_01x02, J3 Screw_Terminal_01x04, J4 Screw_Terminal_01x02, J5 Screw_Terminal_01x02, J6 Screw_Terminal_01x06, J7 Screw_Terminal_01x03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

Commit message: YA AAAAAAAAAAAAAAAA
Detallitos sobre el dxf que estaba mal
Parts:
- removed J1, J10, J2, J4, J9: Screw_Terminal_01x02, TerminalBlock_4Ucon:TerminalBlock_4Ucon_1x02_P3.50mm_Horizontal, symbol Connector:Screw_Terminal_01x02
- added J1, J2, J4, J8, J9: Screw_Terminal_01x03, symbol Connector:Screw_Terminal_01x03
- J12, J3: footprint TerminalBlock_4Ucon:TerminalBlock_4Ucon_1x04_P3.50mm_Horizontal -> (none)
- J5: footprint TerminalBlock_4Ucon:TerminalBlock_4Ucon_1x02_P3.50mm_Horizontal -> (none)
- J6: footprint TerminalBlock_4Ucon:TerminalBlock_4Ucon_1x06_P3.50mm_Horizontal -> (none)
- J7: footprint TerminalBlock_4Ucon:TerminalBlock_4Ucon_1x03_P3.50mm_Horizontal -> (none)
Connections:
- net GND: now also J4.3 (Pin_3), J9.1 (Pin_1)
- net NIVARA_BOARD/DRY_DINPUT_0: now also J4.1 (Pin_1)
- net NIVARA_BOARD/DRY_DINPUT_1: now also J4.2 (Pin_2)
- net NIVARA_BOARD/NPN_DINPUT_0: now also J1.1 (Pin_1)
- net NIVARA_BOARD/NPN_DINPUT_1: now also J1.2 (Pin_2)
- net NIVARA_BOARD/NPN_DOUTPUT_0: now also J8.2 (Pin_2)
- net NIVARA_BOARD/NPN_DOUTPUT_1: now also J8.3 (Pin_3)
- net NIVARA_BOARD/PNP_DINPUT_0: now also J2.1 (Pin_1)
- net NIVARA_BOARD/PNP_DINPUT_1: now also J2.2 (Pin_2)
- net NIVARA_BOARD/PNP_DOUTPUT_0: now also J9.2 (Pin_2)
- net NIVARA_BOARD/PNP_DOUTPUT_1: now also J9.3 (Pin_3)
- net VCC: now also J8.1 (Pin_1)
- net NIVARA_BOARD/mA_AOUTPUT-: no longer names the net of J12.3 (Pin_3)
- new net NPNIN_GND: J1.3 (Pin_3)
- new net PNPIN_GND: J2.3 (Pin_3)
Other:
- sheet NIVARA_BOARD ports: added none; removed mA_AOUTPUT-
- moved on the sheet: AE1, J11, J12, J3, J5, J6, J7
