File: Diseños Kicad/NIVARA CHECK/NIVARA_BOARD.kicad_sch (KiCad schematic)
At the start: 3 parts, among them U1 ESP32-S3-WROOM-1

Commit message: ACTUALIZACION HECHA
PCB SUPUESTA
Parts:
- added R22: 10k, symbol Device:R
- C1: value C -> 1uF
- R1: value R -> 10k
Connections:
- net +3.3V: now also R22.1
- net mA_INTERFAZ_OUT/mA_IN: no longer U1.4 (GPIO4/TOUCH4/ADC1_CH3)
- net ~{RUN}/STOP: now also R22.2
Other:
- sheet NPN_ENTRADA_Mod renamed NPN_IN_Mod
- sheet mA_INTERFAZ_ENTRADA renamed mA_INTERFAZ_IN
- sheet mA_INTERFAZ_SALIDA renamed mA_INTERFAZ_OUT
- added sheet 10V_AIN_INTERFAZ (10V_AIN_INTERFAZ.kicad_sch)
- added sheet 32V_AIN_INTERFAZ (32V_AIN_INTERFAZ.kicad_sch)
- added sheet DRY_INPUT_INTERFAZ (DRY_INPUT_INTERFAZ.kicad_sch)
- added sheet NPN_OUT_INTERFAZ (NPN_OUT_INTERFAZ.kicad_sch)
- added sheet PNP_IN_Mod (PNP_IN_Mod.kicad_sch)
- added sheet PNP_OUT_INTERFAZ (PNP_OUT_INTERFAZ.kicad_sch)
- added sheet VOLTAGE_AOUT_INTERFAZ (VOLTAGE_AOUT_INTERFAZ.kicad_sch)
- sheet NPN_IN_Mod ports: added NPN_Input0, NPN_Input1, NPN_Output0, NPN_Output1; removed none
- sheet RELAY_INTERFAZ: file RELAY_INTERFACE.kicad_sch -> RELAY_INTERFAZ.kicad_sch
- sheet RS485_INTERFAZ: file RS485_INTERFACE.kicad_sch -> RS485_INTERFAZ.kicad_sch
- sheet mA_INTERFAZ_IN: file mA_INTERFACE_IN.kicad_sch -> mA_INTERFAZ_IN.kicad_sch
- sheet mA_INTERFAZ_OUT: file mA_INTERFACE.kicad_sch -> mA_INTERFAZ.kicad_sch
- note added: "NIVARA LA PARA VAMO AVER SI ETO TA BIEN"

Commit message: YA AAAAAAAAAAAAAAAA
Detallitos sobre el dxf que estaba mal
Parts:
- added R31, R32: 4.7k, symbol Device:R
Connections:
- net +3.3V: now also R31.1, R32.1
- net 10V_AIN_INTERFAZ/10V_ADC: now also U1.5 (GPIO5/TOUCH5/ADC1_CH4)
- net 32V_AIN_INTERFAZ/32V_ADC: now also U1.4 (GPIO4/TOUCH4/ADC1_CH3)
- net DRY_INPUT_INTERFAZ/DRY_OUT0: now also U1.18 (GPIO10/TOUCH10/ADC1_CH9/FSPICS0/FSPIIO4/SUBSPICS0)
- net DRY_INPUT_INTERFAZ/DRY_OUT1: now also U1.23 (GPIO21)
- net PNP_IN_Mod/NPN_Output0: now also U1.12 (GPIO8/TOUCH8/ADC1_CH7/SUBSPICS1)
- net PNP_IN_Mod/NPN_Output1: now also U1.17 (GPIO9/TOUCH9/ADC1_CH8/FSPIHD/SUBSPIHD)
- net RS485_INTERFAZ/UART_RX: now also U1.25 (GPIO48/SPICLK_N/SUBSPICLK_N_DIFF); no longer U1.36 (U0RXD/GPIO44/CLK_OUT2)
- net RS485_INTERFAZ/UART_TX: now also U1.24 (GPIO47/SPICLK_P/SUBSPICLK_P_DIFF); no longer U1.37 (U0TXD/GPIO43/CLK_OUT1)
- net RS485_INTERFAZ/~{TRANSMIT}/RECEIVE: now also U1.16 (GPIO46)
- net VOLTAGE_AOUT_INTERFAZ/SCLK: now also U1.8 (GPIO15/U0RTS/ADC2_CH4/XTAL_32K_P), U1.9 (GPIO16/U0CTS/ADC2_CH5/XTAL_32K_N), R31.2, R32.2
- net VOLTAGE_AOUT_INTERFAZ/SEL: now also U1.28 (SPIIO6/GPIO35/FSPID/SUBSPID)
- net ~{RUN}/STOP: now also U1.29 (SPIIO7/GPIO36/FSPICLK/SUBSPICLK)
- net NPN_OUT_INTERFAZ/NPN_EN1: now reaches U1.26 (GPIO45)
- net NPN_OUT_INTERFAZ/NPN_EN0: now reaches U1.31 (GPIO38/FSPIWP/SUBSPIWP)
- net PNP_OUT_INTERFAZ/PNP_EN0: now reaches U1.6 (GPIO6/TOUCH6/ADC1_CH5)
- net PNP_OUT_INTERFAZ/PNP_EN1: now reaches U1.7 (GPIO7/TOUCH7/ADC1_CH6)
Other:
- sheet NPN_OUT_INTERFAZ ports: added NPN_EN0, NPN_EN1; removed NPN_OUT_EN0, NPN_OUT_EN1
- sheet PNP_OUT_INTERFAZ ports: added PNP_EN0, PNP_EN1; removed none
- sheet mA_INTERFAZ_OUT ports: added SCLK, SDA; removed mA_IN, mA_OUT-
- note removed: "NIVARA LA PARA VAMO AVER SI ETO TA BIEN"
- moved on the sheet: C1, R1, R22, U1
