File: Diseños Kicad/NIVARA CHECK/NPN_IN_Mod.kicad_sch (KiCad schematic)
At the start: 6 parts, among them U15 LTV-357TB, U4 LTV-357TB

Commit message: YA AAAAAAAAAAAAAAAA
Detallitos sobre el dxf que estaba mal
Other:
- moved on the sheet: R36, R5, R7, R9, U15, U4
