File: Diseños Kicad/NIVARA CHECK/NPN_OUT_INTERFACE.kicad_sch (KiCad schematic)
At the start: 4 parts

Commit message: YA AAAAAAAAAAAAAAAA
Detallitos sobre el dxf que estaba mal
Other:
- moved on the sheet: R26, R4, U12, U5
