File: Diseños Kicad/NIVARA CHECK/PNP_OUT_INTERFACE.kicad_sch (KiCad schematic)
At the start: 4 parts

Commit message: YA AAAAAAAAAAAAAAAA
Detallitos sobre el dxf que estaba mal
Parts:
- removed R26, R4: 100, symbol Device:R
- removed U12, U5: ~, Package_SO:SO-4_4.4x4.3mm_P2.54mm, symbol Riqi_Parts:GAQY211G2S
- added R29, R30: 100, symbol Device:R
- added U13, U14: ~, Package_SO:SO-4_4.4x4.3mm_P2.54mm, symbol Riqi_Parts:GAQY211G2S
Connections:
- net GND: now also U13.2, U14.2
- new net: R30.2, U14.1
- new net: R29.2, U13.1
- new net PNP_EN0: R29.1
- new net PNP_EN1: R30.1
- new net PNP_OUT0: U13.4
- new net PNP_OUT1: U14.4
- new net VCC: U13.3, U14.3
