File: Diseños Kicad/NIVARA CHECK/PNP_OUT_INTERFAZ.kicad_sch (KiCad schematic)
At the start: 7 parts, among them Q4 NCV8402xST, Q5 NCV8402xST, U13 LTV-357T, U14 LTV-357T

Commit message: YA AAAAAAAAAAAAAAAA
Detallitos sobre el dxf que estaba mal
Parts:
- removed Q4, Q5: NCV8402xST, Package_TO_SOT_SMD:SOT-223, symbol Driver_FET:NCV8402xST
- removed R31: 100, symbol Device:R
- removed R32: R, symbol Device:R
- removed U13, U14: LTV-357T, Package_SO:SO-4_4.4x3.6mm_P2.54mm, symbol Isolator:LTV-357T
- added R30: 100, symbol Device:R
- added U13, U14: ~, Package_SO:SO-4_4.4x4.3mm_P2.54mm, symbol Riqi_Parts:GAQY211G2S
Connections:
- net GND: now also U13.2, U14.2
- net PNP_OUT0: now also U13.4
- net PNP_OUT1: now also U14.4
- net PNP_EN0: now reaches R29.1
- net at R29.2: now also U13.1
- new net: R30.2, U14.1
- new net PNP_EN1: R30.1
- new net VCC: U13.3, U14.3
Other:
- moved on the sheet: R29
