File: Diseños Kicad/NIVARA CHECK/RELAY_INTERFAZ.kicad_sch (KiCad schematic)
At the start: 3 parts, among them K1 G2RL-1, K2 G2RL-1

Commit message: YA AAAAAAAAAAAAAAAA
Detallitos sobre el dxf que estaba mal
Other:
- note removed: "Listo por fiiiiiin"
- moved on the sheet: K1, K2, Q2
