File: Diseños Kicad/NIVARA CHECK/RS485_INTERFACE.kicad_sch (KiCad schematic)
At the start: 4 parts

Commit message: YA AAAAAAAAAAAAAAAA
Detallitos sobre el dxf que estaba mal
Other:
- moved on the sheet: D2, R24, R25, U3
