File: Diseños Kicad/NIVARA CHECK/VOLTAGE_AOUT_INTERFACE.kicad_sch (KiCad schematic)
At the start: 5 parts

Commit message: YA AAAAAAAAAAAAAAAA
Detallitos sobre el dxf que estaba mal
Other:
- moved on the sheet: C7, C8, D3, R23, U11
