File: Diseños Kicad/NIVARA CHECK/mA_INTERFACE.kicad_sch (KiCad schematic)
At the start: 18 parts, among them T1 IRF9310TRPBF

Commit message: YA AAAAAAAAAAAAAAAA
Detallitos sobre el dxf que estaba mal
Other:
- moved on the sheet: C12, C13, C14, C15, D1, D4, D5, JP2, JP3, JP4, R27, R28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
