File: Diseños Kicad/NIVARA CHECK/mA_INTERFACE_IN.kicad_sch (KiCad schematic)
At the start: 2 parts

Commit message: YA AAAAAAAAAAAAAAAA
Detallitos sobre el dxf que estaba mal
Other:
- moved on the sheet: C11, R8
Changed lines of the file:
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@@
 	(generator_version "9.0")
 	(paper "A4")
-	(rectangle
-		(start 19.05 17.78)
-		(end 63.5 55.88)
-		(stroke
-			(width 0)
-			(type default)
-		)
-		(fill
-			(type none)
-		)
-	)
 	(junction
-		(at 33.02 38.1)
+		(at 114.3 100.33)
 		(diameter 0)
 		(color 0 0 0 0)
 	)
 	(junction
-		(at 33.02 29.21)
+		(at 114.3 91.44)
 		(diameter 0)
 		(color 0 0 0 0)
 	)
 	(junction
-		(at 40.64 29.21)
+		(at 121.92 91.44)
 		(diameter 0)
 		(color 0 0 0 0)
@@
 	(wire
 		(pts
-			(xy 33.02 29.21) (xy 33.02 30.48)
-		)
-		(stroke
-			(width 0)
-			(type default)
-		)
-	)
-	(wire
-		(pts
-			(xy 40.64 29.21) (xy 43.18 29.21)
-		)
-		(stroke
-			(width 0)
-			(type default)
-		)
-	)
-	(wire
-		(pts
-			(xy 29.21 29.21) (xy 33.02 29.21)
-		)
-		(stroke
-			(width 0)
-			(type default)
-		)
-	)
-	(wire
-		(pts
-			(xy 33.02 38.1) (xy 40.64 38.1)
-		)
-		(stroke
-			(width 0)
-			(type default)
-		)
-	)
-	(wire
-		(pts
-			(xy 40.64 29.21) (xy 40.64 30.48)
-		)
-		(stroke
-			(width 0)
-			(type default)
-		)
-	)
-	(wire
-		(pts
-			(xy 33.02 29.21) (xy 40.64 29.21)
-		)
-		(stroke
-			(width 0)
-			(type default)
-		)
-	)
-	(wire
-		(pts
-			(xy 33.02 38.1) (xy 33.02 40.64)
+			(xy 114.3 91.44) (xy 114.3 92.71)
+		)
+		(stroke
+			(width 0)
+			(type default)
+		)
+	)
+	(wire
+		(pts
+			(xy 121.92 91.44) (xy 124.46 91.44)
+		)
+		(stroke
+			(width 0)
+			(type default)
+		)
+	)
+	(wire
+		(pts
+			(xy 110.49 91.44) (xy 114.3 91.44)
+		)
+		(stroke
+			(width 0)
+			(type default)
+		)
+	)
+	(wire
+		(pts
+			(xy 114.3 100.33) (xy 121.92 100.33)
+		)
+		(stroke
+			(width 0)
+			(type default)
+		)
+	)
+	(wire
+		(pts
+			(xy 121.92 91.44) (xy 121.92 92.71)
+		)
+		(stroke
+			(width 0)
+			(type default)
+		)
+	)
+	(wire
+		(pts
+			(xy 114.3 91.44) (xy 121.92 91.44)
+		)
+		(stroke
+			(width 0)
+			(type default)
+		)
+	)
+	(wire
+		(pts
+			(xy 114.3 100.33) (xy 114.3 102.87)
 		)
 		(stroke
@@
 	(hierarchical_label "mA_IN"
 		(shape input)
-		(at 29.21 29.21 180)
+		(at 110.49 91.44 180)
 		(effects
 			(font
@@
 	(hierarchical_label "mA_READ"
 		(shape output)
-		(at 43.18 29.21 0)
+		(at 124.46 91.44 0)
 		(effects
 			(font
@@
 	(symbol
 		(lib_id "Device:R")
-		(at 33.02 34.29 180)
+		(at 114.3 96.52 180)
 		(unit 1)
 		(exclude_from_sim no)
@@
 		(fields_autoplaced yes)
 		(property "Reference" "R8"
-			(at 35.56 33.0199 0)
+			(at 116.84 95.2499 0)
 			(effects
 				(font
@@
 		)
 		(property "Value" "120"
-			(at 35.56 35.5599 0)
+			(at 116.84 97.7899 0)
 			(effects
 				(font
@@
 		)
 		(property "Footprint" ""
-			(at 34.798 34.29 90)
+			(at 116.078 96.52 90)
 			(effects
 				(font
@@
 		)
 		(property "Datasheet" "~"
-			(at 33.02 34.29 0)
+			(at 114.3 96.52 0)
 			(effects
 				(font
@@
 		)
 		(property "Description" "Resistor"
-			(at 33.02 34.29 0)
+			(at 114.3 96.52 0)
 			(effects
 				(font
@@
 		)
 		(property "Tolerance" "0.1-1%"
-			(at 33.02 34.29 0)
+			(at 114.3 96.52 0)
 			(effects
 				(font
@@
 		)
 		(instances
-			(project "NIVARA"
+			(project ""
 				(path "/8290cc18-06d0-4e02-a781-29a61ebc321a/9e4d7a0c-a5eb-4e88-9036-0c35e68b279a/89d29688-da71-49bb-a25b-d6f160f4d0d4"
 					(reference "R8")
@@
 	(symbol
 		(lib_id "Device:C")
-		(at 40.64 34.29 0)
+		(at 121.92 96.52 0)
 		(unit 1)
 		(exclude_from_sim no)
@@
 		(fields_autoplaced yes)
 		(property "Reference" "C11"
-			(at 44.45 33.0199 0)
+			(at 125.73 95.2499 0)
 			(effects
 				(font
@@
 		)
 		(property "Value" "100nF"
-			(at 44.45 35.5599 0)
+			(at 125.73 97.7899 0)
 			(effects
 				(font
@@
 		)
 		(property "Footprint" ""
-			(at 41.6052 38.1 0)
+			(at 122.8852 100.33 0)
 			(effects
 				(font
@@
 		)
 		(property "Datasheet" "~"
-			(at 40.64 34.29 0)
+			(at 121.92 96.52 0)
 			(effects
 				(font
@@
 		)
 		(property "Description" "Unpolarized capacitor"
-			(at 40.64 34.29 0)
+			(at 121.92 96.52 0)
 			(effects
 				(font
@@
 	(symbol
 		(lib_id "power:GND")
-		(at 33.02 40.64 0)
+		(at 114.3 102.87 0)
 		(unit 1)
 		(exclude_from_sim no)
@@
 		(fields_autoplaced yes)
 		(property "Reference" "#PWR029"
-			(at 33.02 46.99 0)
+			(at 114.3 109.22 0)
 			(effects
 				(font
@@
 		)
 		(property "Value" "GND"
-			(at 33.02 45.72 0)
+			(at 114.3 107.95 0)
 			(effects
 				(font
@@
 		)
 		(property "Footprint" ""
-			(at 33.02 40.64 0)
+			(at 114.3 102.87 0)
 			(effects
 				(font
@@
 		)
 		(property "Datasheet" ""
-			(at 33.02 40.64 0)
+			(at 114.3 102.87 0)
 			(effects
 				(font
@@
 		)
 		(property "Description" "Power symbol creates a global label with name \"GND\" , ground"
-			(at 33.02 40.64 0)
+			(at 114.3 102.87 0)
 			(effects
 				(font
@@
 		)
 		(instances
-			(project "NIVARA"
+			(project ""
 				(path "/8290cc18-06d0-4e02-a781-29a61ebc321a/9e4d7a0c-a5eb-4e88-9036-0c35e68b279a/89d29688-da71-49bb-a25b-d6f160f4d0d4"
 					(reference "#PWR029")
